File: Kicad/MIDI_to_CV/MIDI_to_CV.sch (KiCad schematic (older format))
At the start: 16 parts, among them IC1 PIC24FJ64GB002-I_SP, J1 Conn_02x08_Odd_Even, J2 PIC Programmer, J3 Panel Connector Male Top, J4 Panel Connector Male Bottom, U1 LD1117S33TR_SOT223, Y1 Crystal

Commit message: Adding lots of decoupling capacitors
Parts:
- added C7, C8: 10uF, symbol Device:CP
Connections:
- net +12V: now also C7.1
- net +5V: now also C8.1
- net GND: now also C7.2, C8.2
Changed lines of the file:
@@
 	1900 1250 1900 1350
 Connection ~ 1900 1250
-Wire Wire Line
-	1900 1250 2150 1250
 Connection ~ 1900 1350
-Wire Wire Line
-	1900 1350 2150 1350
 Wire Wire Line
 	1900 1350 1900 1450
@@
 Connection ~ 2600 1650
 Wire Wire Line
-	2600 1650 3950 1650
+	2600 1650 3000 1650
 $Comp
 L power:PWR_FLAG #FLG0102
@@
 	0    -1   -1   0
 $EndComp
+$Comp
+L Device:CP C8
+U 1 1 5FC85A05
+P 3000 1500
+F 0 "C8" V 3255 1500 50  0000 C CNN
+F 1 "10uF" V 3164 1500 50  0000 C CNN
+F 2 "" H 3038 1350 50  0001 C CNN
+F 3 "~" H 3000 1500 50  0001 C CNN
+	1    3000 1500
+	-1   0    0    1
+$EndComp
+Connection ~ 3000 1650
+Wire Wire Line
+	1900 1350 2150 1350
+Connection ~ 2150 1350
+Wire Wire Line
+	2150 1350 3000 1350
+Wire Wire Line
+	1900 1250 2150 1250
+Wire Wire Line
+	3000 1650 3950 1650
+$Comp
+L Device:CP C7
+U 1 1 5FC9756A
+P 900 1700
+F 0 "C7" V 1155 1700 50  0000 C CNN
+F 1 "10uF" V 1064 1700 50  0000 C CNN
+F 2 "" H 938 1550 50  0001 C CNN
+F 3 "~" H 900 1700 50  0001 C CNN
+	1    900  1700
+	1    0    0    -1
+$EndComp
+Connection ~ 900  1550
+$Comp
+L power:GND #PWR0114
+U 1 1 5FC98A96
+P 900 1850
+F 0 "#PWR0114" H 900 1600 50  0001 C CNN
+F 1 "GND" H 905 1677 50  0000 C CNN
+F 2 "" H 900 1850 50  0001 C CNN
+F 3 "" H 900 1850 50  0001 C CNN
+	1    900  1850
+	1    0    0    -1
+$EndComp
 $EndSCHEMATC
